File: QuickBuckBoard.kicad_pcb (KiCad board)
At the start: 2 copper layers, 14 parts, among them J1 Conn_01x04, J2 Conn_01x04, U1 TI_LM22680QMRE-ADJ

Commit message: First draft layout
Parts:
- removed R4: VISHAYDALE_CRCW12060000Z0EB, Resistors_SMD:R_1206
- added G***: LOGO, DBLS_LOGO:Rooster_4mmx4mm, F.Cu at (74.1, 89.8)
- J1, J2: moved to B.Cu
- moved C2 42.0 mm to (57.0, 80.6), turned to 90 degrees
- moved U1 41.2 mm to (65.0, 81.9), turned to 180 degrees
- moved C3 38.0 mm to (59.7, 80.6), turned to 90 degrees
- moved J1 36.9 mm to (53.3, 86.4)
- moved L1 35.5 mm to (65.4, 89.7)
- moved J2 34.3 mm to (78.7, 86.4)
- moved R3 32.4 mm to (69.2, 78.2)
- moved C5 31.4 mm to (74.3, 82.5), turned to 90 degrees
- moved D1 28.6 mm to (58.4, 87.6), turned to 90 degrees
- moved C4 27.4 mm to (65.0, 85.3)
- moved R1 27.2 mm to (69.6, 80.7), turned to 270 degrees
- moved R2 23.5 mm to (67.0, 78.3), turned to 180 degrees
- moved C1 21.0 mm to (69.6, 83.1), turned to 270 degrees
Connections:
- C5 pad 1: Net-(C5-Pad1) -> +5V
- L1 pad 2: Net-(C5-Pad1) -> +5V
- R3 pad 2: Net-(C5-Pad1) -> +5V
Routing:
- net GND: track 0.00 -> 17.1 mm, vias 0 -> 25
- net /5V_ENABLE: track 0.00 -> 12.7 mm
- net Net-(C4-Pad1): track 0.00 -> 9.17 mm
- net +5V: track 0.00 -> 6.66 mm
- net Net-(R2-Pad1): track 0.00 -> 3.18 mm
- net Net-(C4-Pad2): track 0.00 -> 3.08 mm
- net Net-(R1-Pad2): track 0.00 -> 2.18 mm
- net Net-(C1-Pad1): track 0.00 -> 2.08 mm
- added copper zone on F.Cu, net +5V
- added copper zone on B.Cu, net GND
- added copper zone on F.Cu, net GND
- added copper zone on F.Cu, net Net-(C4-Pad1)
- added copper zone on F.Cu, net VBUS
Other:
- board outline added: 30.5 x 17.1 mm
- net class Default: clearance 0.2 -> 0.2032; trace_width 0.25 -> 0.254; via_dia 0.8 -> 0.8128; via_drill 0.4 -> 0.381
- rule trace_clearance: 0.2 -> 0.2032
- rule trace_min: 0.2 -> 0.2032
- rule via_min_drill: 0.3 -> 0.381
- rule via_min_size: 0.4 -> 0.635
- board text added: "Dirtbag Lab Supplies"
- board text added: "EN"
- board text added: "GND"
- board text added: "Quick Buck v1.0"
- board text added: "VIN"
- board text added: "VOUT"
