File: QuickBuckBoard.sch (KiCad schematic (older format))
At the start: 14 parts, among them J1 Conn_01x04, J2 Conn_01x04, U1 TI_LM22680QMRE-ADJ

Commit message: First draft layout
Parts:
- removed R4: VISHAYDALE_CRCW12060000Z0EB, Resistors_SMD:R_1206, symbol DBLS_Resistor:VISHAYDALE_CRCW12060000Z0EB
Connections:
- net +5V: now also C5.1, L1.2, R3.2
Changed lines of the file:
@@
 $EndDescr
-$Comp
-L DBLS_Resistor:VISHAYDALE_CRCW12060000Z0EB R4
-U 1 1 615EC717
-P 7200 4600
-F 0 "R4" H 7250 4650 45  0000 L BNN
-F 1 "VISHAYDALE_CRCW12060000Z0EB" H 6800 5250 50  0001 L BNN
-F 2 "Resistors_SMD:R_1206" H 7200 4800 50  0001 C CNN
-F 3 "N/A" H 7200 4800 50  0001 C CNN
-F 4 "0R" H 7200 4540 40  0000 C CNN "resistance"
-F 5 "Vishay Dale" H 7200 5200 50  0001 C CNN "mfg"
-F 6 "CRCW12060000Z0EB" H 7200 5100 50  0001 C CNN "mfg_pn"
-F 7 "Digikey" H 7200 5000 50  0001 C CNN "vendor"
-F 8 "541-3032-1-ND" H 7200 4900 50  0001 C CNN "vendor_pn"
-F 9 "YES" H 7100 4650 20  0001 C CNN "place"
-	1    7200 4600
-	1    0    0    -1
-$EndComp
-Wire Wire Line
-	6900 4600 7100 4600
 $Comp
 L power:+5V #PWR0101
@@
 Wire Wire Line
 	7500 4550 7500 4600
-Wire Wire Line
-	7300 4600 7500 4600
 Connection ~ 7500 4600
 Wire Wire Line
@@
 	1    0    0    -1
 $EndComp
+Wire Wire Line
+	6900 4600 7500 4600
 $EndSCHEMATC
